Commit message: Barebones URDF parsing on a test UR5e URDF file
* More work is needed to add collision data in lieu of inertial data to ur5 URDF
* More work is needed to handle collision geometry in parser

File: referenceframe/testurdf/ur5.urdf (robot description, URDF)
Before this commit: robot ur5, 9 links, 8 joints
Links:
- link base_link: mass 4.0 -> None
- link link1: mass 3.7 -> None
- link link2: mass 8.393 -> None
- link link3: mass 2.275 -> None
- link link4: mass 1.219 -> None
- link link5: mass 1.219 -> None
- link link6: mass 0.1879 -> None

Commit message: Responding to draft PR comments, some small optimizations

File: referenceframe/testurdf/ur5.urdf (robot description, URDF)
Before this commit: robot ur5, 9 links, 8 joints
Links:
- link base_link: geometry collision sphere radius=0.001
- link link1: geometry collision sphere radius=0.001
- link link2: geometry collision sphere radius=0.001
- link link3: geometry collision sphere radius=0.001
- link link4: geometry collision sphere radius=0.001
- link link5: geometry collision sphere radius=0.001
- link link6: geometry collision sphere radius=0.001
